File: elec/layout/default/usbc.kicad_pcb (KiCad board)
At the start: 2 copper layers, 225.7 x 100.8 mm, 3 parts

Commit message: Remove junk from layout
Other:
- board outline removed
- board text removed: "{{GITHASH}}"
